Commit message: Change model of drone and move sensors

File: hector_quadrotor_description/urdf/quadrotor_base.urdf.xacro (robot description, xacro)
@@ -12,34 +12,34 @@
       </inertial>
       <visual>
-        <origin xyz="0 0 0" rpy="0 0 0" />
+        <origin xyz="0 0 0" rpy="${pi/2} 0 ${pi/2}" />
         <geometry>
-          <mesh filename="package://hector_quadrotor_description/meshes/quadrotor/quadrotor_base.dae"/>
+          <mesh filename="package://hector_quadrotor_description/meshes/quadrotor/tiltrotor.stl"/>
         </geometry>
       </visual>
       <collision>
-        <origin xyz="0 0 0" rpy="0 0 0" />
+        <origin xyz="0 0 0" rpy="${pi/2} 0 ${pi/2}" />
         <geometry>
-          <mesh filename="package://hector_quadrotor_description/meshes/quadrotor/quadrotor_base.stl"/>
+          <mesh filename="package://hector_quadrotor_description/meshes/quadrotor/tiltrotor.stl"/>
         </geometry>
       </collision>
      </link>
      <!-- Left = RED -->
-     <xacro:sonar_sensor name="sonar_right" parent="base_link" ros_topic="sonar_right" update_rate="10" min_range="0.03" max_range="10.0" field_of_view="${3*pi/180}" ray_count="3">
-        <origin xyz="-0.06 0.0 0.05" rpy="0 0 ${180*pi/180}"/>
+     <xacro:sonar_sensor name="sonar_backward" parent="base_link" ros_topic="sonar_backward" update_rate="10" min_range="0.03" max_range="10.0" field_of_view="${3*pi/180}" ray_count="3">
+        <origin xyz="-0.315 0.0 0.035" rpy="0 0 ${180*pi/180}"/>
+      </xacro:sonar_sensor>
+      <xacro:sonar_sensor name="sonar_forward" parent="base_link" ros_topic="sonar_forward" update_rate="10" min_range="0.03" max_range="10.0" field_of_view="${3*pi/180}" ray_count="3">
+        <origin xyz="0.325 0.0 -0.05" rpy="0 0 0"/>
       </xacro:sonar_sensor>
       <xacro:sonar_sensor name="sonar_left" parent="base_link" ros_topic="sonar_left" update_rate="10" min_range="0.03" max_range="10.0" field_of_view="${3*pi/180}" ray_count="3">
-        <origin xyz="0.06 0.0 0.05" rpy="0 0 0"/>
+        <origin xyz="0.0 0.06 -0.03" rpy="0 0 ${90*pi/180}"/>
       </xacro:sonar_sensor>
-      <xacro:sonar_sensor name="sonar_backward" parent="base_link" ros_topic="sonar_backward" update_rate="10" min_range="0.03" max_range="10.0" field_of_view="${3*pi/180}" ray_count="3">
-        <origin xyz="0.0 0.06 0.05" rpy="0 0 ${90*pi/180}"/>
-      </xacro:sonar_sensor>
-      <xacro:sonar_sensor name="sonar_forward" parent="base_link" ros_topic="sonar_forward" update_rate="10" min_range="0.03" max_range="10.0" field_of_view="${3*pi/180}" ray_count="3">
-        <origin xyz="0.0 -0.06 0.05" rpy="0 0 ${-90*pi/180}"/>
+      <xacro:sonar_sensor name="sonar_right" parent="base_link" ros_topic="sonar_right" update_rate="10" min_range="0.03" max_range="10.0" field_of_view="${3*pi/180}" ray_count="3">
+        <origin xyz="0.0 -0.06 -0.03" rpy="0 0 ${-90*pi/180}"/>
       </xacro:sonar_sensor>
       <xacro:sonar_sensor name="sonar_up" parent="base_link" ros_topic="sonar_up" update_rate="10" min_range="0.03" max_range="10.0" field_of_view="${3*pi/180}" ray_count="3">
-        <origin xyz="0.0 0.0 0.04" rpy="0 ${-90*pi/180} 0"/>
+        <origin xyz="-0.24 0.0 0.05" rpy="0 ${-90*pi/180} 0"/>
       </xacro:sonar_sensor>
       <xacro:sonar_sensor name="sonar_down" parent="base_link" ros_topic="sonar_down" update_rate="10" min_range="0.03" max_range="10.0" field_of_view="${3*pi/180}" ray_count="3">
-        <origin xyz="0.0 0.0 -0.13" rpy="0 ${90*pi/180} 0"/>
+        <origin xyz="0.0 0.0 -0.05" rpy="0 ${90*pi/180} 0"/>
       </xacro:sonar_sensor>
   </xacro:macro>

File: hector_quadrotor_description/urdf/quadrotor_hokuyo_utm30lx.urdf.xacro (robot description, xacro)
@@ -10,8 +10,8 @@
     <xacro:quadrotor_base_macro />
     <!-- Hokuyo UTM-30LX mounted upside down below the quadrotor body -->
-    <xacro:include filename="$(find hector_sensors_description)/urdf/hokuyo_utm30lx.urdf.xacro" />
+    <!--<xacro:include filename="$(find hector_sensors_description)/urdf/hokuyo_utm30lx.urdf.xacro" />
     <xacro:hokuyo_utm30lx name="laser0" parent="base_link" ros_topic="scan" update_rate="40" ray_count="1081" min_angle="-135" max_angle="135">
       <origin xyz="0.0 0.0 -0.097" rpy="${M_PI} 0 0"/>
-    </xacro:hokuyo_utm30lx>
+    </xacro:hokuyo_utm30lx>-->
     <!-- Forward facing camera -->
     <xacro:include filename="$(find hector_sensors_description)/urdf/generic_camera.urdf.xacro" />

File: hector_quadrotor_description/urdf/quadrotor_with_asus_with_hokuyo_utm30lx.urdf.xacro (robot description, xacro)
@@ -10,12 +10,12 @@
     <xacro:quadrotor_base_macro />
     <!-- Hokuyo UTM-30LX mounted upside down below the quadrotor body -->
-    <xacro:include filename="$(find hector_sensors_description)/urdf/hokuyo_utm30lx.urdf.xacro" />
+    <!--<xacro:include filename="$(find hector_sensors_description)/urdf/hokuyo_utm30lx.urdf.xacro" />
     <xacro:hokuyo_utm30lx name="laser0" parent="base_link" ros_topic="scan" update_rate="40" ray_count="1081" min_angle="-135" max_angle="135">
       <origin xyz="0.0 0.0 -0.097" rpy="${M_PI} 0 0"/>
     </xacro:hokuyo_utm30lx>
-    <!-- Asus Xiton Live Pro -->
+    <!-- Asus Xiton Live Pro --
     <xacro:include filename="$(find hector_sensors_description)/urdf/asus_camera.urdf.xacro" />
     <xacro:asus_camera name="camera" parent="base_link">
       <origin xyz="0.1 0.0 -0.03" rpy="0 ${M_PI/9} 0"/>
-    </xacro:asus_camera>
+    </xacro:asus_camera>-->
 </robot>

File: hector_quadrotor_description/urdf/quadrotor_with_cam.urdf.xacro (robot description, xacro)
@@ -10,7 +10,7 @@
     <xacro:quadrotor_base_macro />
     <!-- Forward facing camera -->
-    <xacro:include filename="$(find hector_sensors_description)/urdf/generic_camera.urdf.xacro" />
+    <!--<xacro:include filename="$(find hector_sensors_description)/urdf/generic_camera.urdf.xacro" />
     <xacro:generic_camera name="front_cam" parent="base_link" ros_topic="camera/image" cam_info_topic="camera/camera_info" update_rate="10" res_x="320" res_y="240" image_format="R8G8B8" hfov="90">
       <origin xyz="0.05 0.0 -0.06" rpy="0 0 0"/>
-    </xacro:generic_camera>
+    </xacro:generic_camera>-->
 </robot>

Commit message: Add Maarten's changes.

File: hector_quadrotor_description/urdf/quadrotor_base.urdf.xacro (robot description, xacro)
@@ -1,4 +1,4 @@
 <?xml version="1.0"?>
-<robot xmlns:xacro="http://ros.org/wiki/xacro">
+<robot name="quadrotor" xmlns:xacro="http://ros.org/wiki/xacro">
   <xacro:include filename="$(find hector_sensors_description)/urdf/sonar_sensor.urdf.xacro" />
   <xacro:property name="pi" value="3.1415926535897931" />
@@ -6,5 +6,5 @@
   <xacro:macro name="quadrotor_base_macro">
     <link name="base_link">
-     <inertial>
+      <inertial>
         <mass value="1.477" />
         <origin xyz="0 0 0" />
@@ -12,18 +12,18 @@
       </inertial>
       <visual>
-        <origin xyz="0 0 0" rpy="0 0 0" />
+        <origin xyz="0 0 0" rpy="${pi/2} 0 ${pi/2}" />
         <geometry>
-          <mesh filename="package://hector_quadrotor_description/meshes/quadrotor/quadrotor_base.dae"/>
+          <mesh filename="package://hector_quadrotor_description/meshes/quadrotor/quadcopter.stl"/>
         </geometry>
       </visual>
       <collision>
-        <origin xyz="0 0 0" rpy="0 0 0" />
+        <origin xyz="0 0 0" rpy="${pi/2} 0 ${pi/2}" />>
         <geometry>
-          <mesh filename="package://hector_quadrotor_description/meshes/quadrotor/quadrotor_base.stl"/>
+          <mesh filename="package://hector_quadrotor_description/meshes/quadrotor/quadcopter.stl"/>
         </geometry>
       </collision>
-     </link>
-     <!-- Left = RED -->
-     <xacro:sonar_sensor name="sonar_right" parent="base_link" ros_topic="sonar_right" update_rate="10" min_range="0.03" max_range="10.0" field_of_view="${3*pi/180}" ray_count="3">
+    </link>
+    <!-- Sonar height sensors -->
+    <xacro:sonar_sensor name="sonar_right" parent="base_link" ros_topic="sonar_right" update_rate="10" min_range="0.03" max_range="10.0" field_of_view="${3*pi/180}" ray_count="3">
         <origin xyz="-0.06 0.0 0.05" rpy="0 0 ${180*pi/180}"/>
       </xacro:sonar_sensor>

Commit message: New model with landing gear and updated sensor positions

File: hector_quadrotor_description/urdf/quadrotor_base.urdf.xacro (robot description, xacro)
@@ -7,7 +7,7 @@
     <link name="base_link">
      <inertial>
-        <mass value="1.477" />
+        <mass value="3.8" />
         <origin xyz="0 0 0" />
-        <inertia ixx="0.01152" ixy="0.0" ixz="0.0" iyy="0.01152" iyz="0.0" izz="0.0218" />
+        <inertia ixx="-0.0888" ixy="-0.000207" ixz="0" iyy="0.132" iyz="0.000574" izz="0.0694" />
       </inertial>
       <visual>
@@ -38,8 +38,8 @@
       </xacro:sonar_sensor>
       <xacro:sonar_sensor name="sonar_up" parent="base_link" ros_topic="sonar_up" update_rate="10" min_range="0.03" max_range="10.0" field_of_view="${3*pi/180}" ray_count="3">
-        <origin xyz="-0.24 0.0 0.05" rpy="0 ${-90*pi/180} 0"/>
+        <origin xyz="0.27 0.0 0.04" rpy="0 ${-90*pi/180} 0"/>
       </xacro:sonar_sensor>
       <xacro:sonar_sensor name="sonar_down" parent="base_link" ros_topic="sonar_down" update_rate="10" min_range="0.03" max_range="10.0" field_of_view="${3*pi/180}" ray_count="3">
-        <origin xyz="0.0 0.0 -0.05" rpy="0 ${90*pi/180} 0"/>
+        <origin xyz="0.29 0.0 -0.07" rpy="0 ${90*pi/180} 0"/>
       </xacro:sonar_sensor>
   </xacro:macro>
